File: PCB/KB-Starter.kicad_sch (KiCad schematic)
At the start: 67 parts, among them J1 USB_C_Receptacle_USB2.0, J2 SWD, SW1 SW_Push, U1 W25Q128JVS, U2 USBLC6-2SC6, U3 XC6206PxxxMR, U5 RP2040, Y1 12MHz

Commit message: fix+feat: matrix fix + touchup
Parts:
- SW1: footprint Connector_PinSocket_2.54mm:PinSocket_1x02_P2.54mm_Vertical -> Button_Switch_SMD:SW_SPST_FSMSM
Connections:
- net GPIO5 is gone; now on net COL1: U5.7 (GPIO5)
- net COL1: no longer U5.8 (GPIO6)
- net COL2: now also U5.8 (GPIO6); no longer U5.9 (GPIO7)
- net COL3: now also U5.9 (GPIO7); no longer U5.11 (GPIO8)
- net COL4: now reaches MX15.2, MX4.2, MX8.2
- net COL4: now also U5.11 (GPIO8)
- no-connect marks 24 -> 23
Changed lines of the file:
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@@
   (junction (at 139.7 142.24) (diameter 0) (color 0 0 0 0)
+  )
+  (junction (at 165.1 99.06) (diameter 0) (color 0 0 0 0)
   )
   (junction (at 214.63 85.09) (diameter 0) (color 0 0 0 0)
@@
   (no_connect (at 257.81 55.88))
   (no_connect (at 187.96 120.65))
-  (no_connect (at 187.96 123.19))
   (no_connect (at 187.96 156.21))
   (no_connect (at 187.96 146.05))
@@
   (no_connect (at 220.98 115.57))
   (no_connect (at 220.98 110.49))
+  (wire (pts (xy 165.1 90.17) (xy 165.1 99.06))
+    (stroke (width 0) (type default))
+  )
   (wire (pts (xy 90.17 81.28) (xy 85.09 81.28))
     (stroke (width 0) (type default))
@@
     (stroke (width 0) (type default))
   )
-  (wire (pts (xy 190.5 128.27) (xy 187.96 128.27))
+  (wire (pts (xy 187.96 125.73) (xy 190.5 125.73))
     (stroke (width 0) (type default))
   )
@@
     (stroke (width 0) (type default))
   )
+  (wire (pts (xy 190.5 128.27) (xy 187.96 128.27))
+    (stroke (width 0) (type default))
+  )
   (wire (pts (xy 181.61 62.23) (xy 184.15 62.23))
     (stroke (width 0) (type default))
@@
   )
   (wire (pts (xy 238.76 92.71) (xy 238.76 91.44))
+    (stroke (width 0) (type default))
+  )
+  (wire (pts (xy 187.96 130.81) (xy 190.5 130.81))
     (stroke (width 0) (type default))
   )
@@
     (stroke (width 0) (type default))
   )
-  (wire (pts (xy 190.5 130.81) (xy 187.96 130.81))
-    (stroke (width 0) (type default))
-  )
   (wire (pts (xy 85.09 73.66) (xy 90.17 73.66))
     (stroke (width 0) (type default))
@@
     (stroke (width 0) (type default))
   )
-  (wire (pts (xy 190.5 125.73) (xy 187.96 125.73))
-    (stroke (width 0) (type default))
-  )
   (wire (pts (xy 109.22 106.68) (xy 124.46 106.68))
     (stroke (width 0) (type default))
@@
     (stroke (width 0) (type default))
   )
+  (wire (pts (xy 190.5 123.19) (xy 187.96 123.19))
+    (stroke (width 0) (type default))
+  )
   (wire (pts (xy 85.09 58.42) (xy 90.17 58.42))
     (stroke (width 0) (type default))
@@
     )
   )
-  (global_label "COL3" (shape input) (at 190.5 130.81 0) (fields_autoplaced)
+  (global_label "COL3" (shape input) (at 190.5 128.27 0) (fields_autoplaced)
+    (effects (font (size 1.27 1.27)) (justify left))
+    (property "Intersheetrefs" "${INTERSHEET_REFS}" (at 198.2439 128.27 0)
+      (effects (font (size 1.27 1.27)) (justify left) hide)
+    )
+  )
+  (global_label "ROW4" (shape input) (at 167.64 160.02 0) (fields_autoplaced)
+    (effects (font (size 1.27 1.27)) (justify left))
+    (property "Intersheetrefs" "${INTERSHEET_REFS}" (at 175.8072 160.02 0)
+      (effects (font (size 1.27 1.27)) (justify left) hide)
+    )
+  )
+  (global_label "D_N" (shape input) (at 24.13 40.64 180) (fields_autoplaced)
+    (effects (font (size 1.27 1.27)) (justify right))
+    (property "Intersheetrefs" "${INTERSHEET_REFS}" (at 18.1488 40.5606 0)
+      (effects (font (size 1.27 1.27)) (justify right) hide)
+    )
+  )
+  (global_label "D_USB_N" (shape input) (at 213.36 30.48 0) (fields_autoplaced)
+    (effects (font (size 1.27 1.27)) (justify left))
+    (property "Intersheetrefs" "${INTERSHEET_REFS}" (at 224.1188 30.4006 0)
+      (effects (font (size 1.27 1.27)) (justify left) hide)
+    )
+  )
+  (global_label "ROW2" (shape input) (at 190.5 135.89 0) (fields_autoplaced)
+    (effects (font (size 1.27 1.27)) (justify left))
+    (property "Intersheetrefs" "${INTERSHEET_REFS}" (at 198.6672 135.89 0)
+      (effects (font (size 1.27 1.27)) (justify left) hide)
+    )
+  )
+  (global_label "XTAL_IN" (shape input) (at 213.36 57.15 0) (fields_autoplaced)
+    (effects (font (size 1.27 1.27)) (justify left))
+    (property "Intersheetrefs" "${INTERSHEET_REFS}" (at 222.9698 57.0706 0)
+      (effects (font (size 1.27 1.27)) (justify left) hide)
+    )
+  )
+  (global_label "XTAL_OUT" (shape input) (at 34.29 86.36 180) (fields_autoplaced)
+    (effects (font (size 1.27 1.27)) (justify right))
+    (property "Intersheetrefs" "${INTERSHEET_REFS}" (at 22.9869 86.2806 0)
+      (effects (font (size 1.27 1.27)) (justify right) hide)
+    )
+  )
+  (global_label "D_USB_P" (shape input) (at 257.81 48.26 0) (fields_autoplaced)
+    (effects (font (size 1.27 1.27)) (justify left))
+    (property "Intersheetrefs" "${INTERSHEET_REFS}" (at 268.5083 48.3394 0)
+      (effects (font (size 1.27 1.27)) (justify left) hide)
+    )
+  )
+  (global_label "COL4" (shape input) (at 190.5 130.81 0) (fields_autoplaced)
     (effects (font (size 1.27 1.27)) (justify left))
     (property "Intersheetrefs" "${INTERSHEET_REFS}" (at 198.2439 130.81 0)
@@
     )
   )
-  (global_label "ROW4" (shape input) (at 167.64 160.02 0) (fields_autoplaced)
-    (effects (font (size 1.27 1.27)) (justify left))
-    (property "Intersheetrefs" "${INTERSHEET_REFS}" (at 175.8072 160.02 0)
-      (effects (font (size 1.27 1.27)) (justify left) hide)
-    )
-  )
-  (global_label "D_N" (shape input) (at 24.13 40.64 180) (fields_autoplaced)
-    (effects (font (size 1.27 1.27)) (justify right))
-    (property "Intersheetrefs" "${INTERSHEET_REFS}" (at 18.1488 40.5606 0)
-      (effects (font (size 1.27 1.27)) (justify right) hide)
-    )
-  )
-  (global_label "D_USB_N" (shape input) (at 213.36 30.48 0) (fields_autoplaced)
-    (effects (font (size 1.27 1.27)) (justify left))
-    (property "Intersheetrefs" "${INTERSHEET_REFS}" (at 224.1188 30.4006 0)
-      (effects (font (size 1.27 1.27)) (justify left) hide)
-    )
-  )
-  (global_label "ROW2" (shape input) (at 190.5 135.89 0) (fields_autoplaced)
-    (effects (font (size 1.27 1.27)) (justify left))
-    (property "Intersheetrefs" "${INTERSHEET_REFS}" (at 198.6672 135.89 0)
-      (effects (font (size 1.27 1.27)) (justify left) hide)
-    )
-  )
-  (global_label "XTAL_IN" (shape input) (at 213.36 57.15 0) (fields_autoplaced)
-    (effects (font (size 1.27 1.27)) (justify left))
-    (property "Intersheetrefs" "${INTERSHEET_REFS}" (at 222.9698 57.0706 0)
-      (effects (font (size 1.27 1.27)) (justify left) hide)
-    )
-  )
-  (global_label "XTAL_OUT" (shape input) (at 34.29 86.36 180) (fields_autoplaced)
-    (effects (font (size 1.27 1.27)) (justify right))
-    (property "Intersheetrefs" "${INTERSHEET_REFS}" (at 22.9869 86.2806 0)
-      (effects (font (size 1.27 1.27)) (justify right) hide)
-    )
-  )
-  (global_label "D_USB_P" (shape input) (at 257.81 48.26 0) (fields_autoplaced)
-    (effects (font (size 1.27 1.27)) (justify left))
-    (property "Intersheetrefs" "${INTERSHEET_REFS}" (at 268.5083 48.3394 0)
-      (effects (font (size 1.27 1.27)) (justify left) hide)
-    )
-  )
   (global_label "SD1" (shape input) (at 34.29 55.88 180) (fields_autoplaced)
     (effects (font (size 1.27 1.27)) (justify right))
@@
     )
   )
-  (global_label "COL2" (shape input) (at 190.5 128.27 0) (fields_autoplaced)
-    (effects (font (size 1.27 1.27)) (justify left))
-    (property "Intersheetrefs" "${INTERSHEET_REFS}" (at 198.2439 128.27 0)
+  (global_label "COL2" (shape input) (at 190.5 125.73 0) (fields_autoplaced)
+    (effects (font (size 1.27 1.27)) (justify left))
+    (property "Intersheetrefs" "${INTERSHEET_REFS}" (at 198.2439 125.73 0)
       (effects (font (size 1.27 1.27)) (justify left) hide)
     )
@@
     )
   )
+  (global_label "COL4" (shape input) (at 165.1 90.17 90) (fields_autoplaced)
+    (effects (font (size 1.27 1.27)) (justify left))
+    (property "Intersheetrefs" "${INTERSHEET_REFS}" (at 165.1 82.4261 90)
+      (effects (font (size 1.27 1.27)) (justify left) hide)
+    )
+  )
   (global_label "D_USB_N" (shape input) (at 257.81 43.18 0) (fields_autoplaced)
     (effects (font (size 1.27 1.27)) (justify left))
@@
     )
   )
-  (global_label "COL1" (shape input) (at 190.5 125.73 0) (fields_autoplaced)
-    (effects (font (size 1.27 1.27)) (justify left))
-    (property "Intersheetrefs" "${INTERSHEET_REFS}" (at 198.2439 125.73 0)
-      (effects (font (size 1.27 1.27)) (justify left) hide)
-    )
-  )
   (global_label "QSPI_CLK" (shape input) (at 34.29 63.5 180) (fields_autoplaced)
     (effects (font (size 1.27 1.27)) (justify right))
@@
     (property "Intersheetrefs" "${INTERSHEET_REFS}" (at 135.6452 34.29 0)
       (effects (font (size 1.27 1.27)) (justify right) hide)
+    )
+  )
+  (global_label "COL1" (shape input) (at 190.5 123.19 0) (fields_autoplaced)
+    (effects (font (size 1.27 1.27)) (justify left))
+    (property "Intersheetrefs" "${INTERSHEET_REFS}" (at 198.2439 123.19 0)
+      (effects (font (size 1.27 1.27)) (justify left) hide)
     )
   )
@@
       (effects (font (size 1.27 1.27)))
     )
-    (property "Footprint" "Connector_PinSocket_2.54mm:PinSocket_1x02_P2.54mm_Vertical" (at 119.38 19.05 0)
-      (effects (font (size 1.27 1.27)) hide)
-    )
+    (property "Footprint" "Button_Switch_SMD:SW_SPST_FSMSM" (at 119.38 19.05 0)
+      (effects (font (size 1.27 1.27)) hide)
+    )

Commit message: add missing 3d models, cleanup for KiCad 8, swd
Parts:
- removed J2: SWD, Connector_PinSocket_2.54mm:PinSocket_1x05_P2.54mm_Vertical, symbol Connector_Generic:Conn_01x05
- added J2: 3-pin SWD, Connector_JST:JST_SH_SM03B-SRSS-TB_1x03-1MP_P1.00mm_Horizontal, symbol Connector:Conn_01x03_Socket
- D1, D10, D11, D12, D13, D14, D15, D16, D17, D2, D3, D4, D5, D6, D7, D8, D9: LCSC (none) -> C727112
- MX1, MX10, MX11, MX13, MX14, MX17, MX2, MX3, MX4, MX5, MX6, MX7, MX9: value SW_Push -> Kailh Hotswap; LCSC (none) -> C5156480
- MX12, MX15, MX8: value SW_Push -> Kailh Hotswap; footprint PCM_Switch_Keyboard_Hotswap_Kailh:SW_Hotswap_Kailh_MX_2.00u_90deg -> PCM_Switch_Keyboard_Hotswap_Kailh:SW_Hotswap_Kailh_MX_1.00u; LCSC (none) -> C5156480
- MX16: value SW_Push -> Kailh Hotswap; footprint PCM_Switch_Keyboard_Hotswap_Kailh:SW_Hotswap_Kailh_MX_2.00u -> PCM_Switch_Keyboard_Hotswap_Kailh:SW_Hotswap_Kailh_MX_1.00u; LCSC (none) -> C5156480
- SW1: footprint Button_Switch_SMD:SW_SPST_FSMSM -> Button_Switch_SMD:SW_SPST_PTS810; LCSC (none) -> C221896
- U3: LCSC (none) -> C5250982
- U5: LCSC (none) -> C2040
Connections:
- net GND: now also J2.2 (Pin_2)
- net SWCLK: now also J2.3 (Pin_3)
- net SWD: now also J2.1 (Pin_1)

Commit message: feat: cleanup, graphics, JLCPCB DRU
Parts:
- removed J2: 3-pin SWD, Connector_JST:JST_SH_SM03B-SRSS-TB_1x03-1MP_P1.00mm_Horizontal, symbol Connector:Conn_01x03_Socket
- added J2: 3-pin SWD, Connector_JST:JST_SH_BM03B-SRSS-TB_1x03-1MP_P1.00mm_Vertical, symbol Connector_Generic_MountingPin:Conn_01x03_MountingPin
- added J3: 3-pin UART, Connector_JST:JST_SH_BM03B-SRSS-TB_1x03-1MP_P1.00mm_Vertical, symbol Connector_Generic_MountingPin:Conn_01x03_MountingPin
- added R10, R11, R8, R9: 100, Resistor_SMD:R_0603_1608Metric, symbol Device:R
Connections:
- net GND: now also J2.2 (Pin_2), J2.MP (MountPin), J3.2 (Pin_2), J3.MP (MountPin)
- net SWCLK: now also R10.1
- net SWD: now also R11.1
- net GPIO20 renamed UART0_TX
- net UART0_TX: now also R8.1
- net GPIO21 renamed UART0_RX
- net UART0_RX: now also R9.2
- new net: J2.1 (Pin_1), R10.2
- new net: J2.3 (Pin_3), R11.2
- new net: J3.1 (Pin_1), R8.2
- new net: J3.3 (Pin_3), R9.1
- no-connect marks 23 -> 2
Other:
- note added: "DECOUPLING"
- note added: "ESD"
- note added: "FLASH"
- note added: "IO"
- note added: "LDO"
- note added: "MATRIX"
- note added: "OSCILLATOR"
- note added: "RP2040"
- note added: "SWD JST"
- note added: "UART JST"
- note added: "USB"
- moved on the sheet: C16, D1, D10, D11, D12, D13, D14, D15, D16, D17, D2, D3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
